File: pcb-layout/controller.brd (EAGLE design)
At the start: 38 x 35.5 mm, 21 parts, among them IC1 MEGA48/88/168-AU, J1 AVR_SPI_PRG_6PTH

Commit message: Updated board to fix a number of problems
* Used DMN53D0LW layout for the DMN6140L part which has a smaller footprint. Created a new layout for DMN6140L and used that
* Removed resistor in series with flyback diode.
* Updated diode layout to be 1N4004 compatible
* Removed diode across FET (was there assuming it would be a BJT)
* Fixed reset resistor, attaching it to VCC rather than GND
* Added a cap from reset to ground
* Fixed motor PWM output pin from ADC6 (not for pwm output) to ADC0
Parts:
- removed D1: (no value), SparkFun:DIODE-1N4001
- removed MOTOR-BAD_FOOTPRINT: DMN53D0LW, GARTH:SOT-323
- removed R1: (no value), SparkFun:1206
- added D2: 1N4004, diode:DO41-10
- U$2: value DIODE-ZENERPTH -> DMN6140L; device SparkFun:DIODE-ZENER -> GARTH:SOT-32-DIODES
- moved C6 38.0 mm to (15.7, 27.4)
- moved U$2 1.27 mm to (24.1, 7.62), turned to 0 degrees
Connections:
- removed net N$1: D1.A, R1.2
- removed net V5: R3.1
- net 12V: now also D2.C; no longer D1.C
- net 5V: now also R3.1
- net GND: now also U$2.S; no longer MOTOR-BAD_FOOTPRINT.P$3, U$2.P$2
- net MOTOR-: now also D2.A, U$2.D; no longer MOTOR-BAD_FOOTPRINT.P$1, R1.1, U$2.P$1
- net MOTOR_CTRL: now also U$2.G; no longer MOTOR-BAD_FOOTPRINT.P$2
Routing:
- net GND: track 122.9 -> 97.0 mm
- net MOTOR_CTRL: track 15.1 -> 23.9 mm, vias 0 -> 2
- net 5V: track 52.0 -> 58.6 mm, vias 2 -> 3
- net RESET: track 10.3 -> 12.8 mm
- net N$1: track 2.41 -> 0.00 mm
- net MOTOR-: track 12.0 -> 10.4 mm
Other:
- board text added: "2019-02-06"
- board text added: "Grinder Controller v2"
- board text removed: "2018-02-11"
- board text removed: "Grinder Controller v1"
