File: pcb-layout/controller.sch (EAGLE design)
At the start: 21 parts, among them IC1 MEGA48/88/168-AU, J1 AVR_SPI_PRG_6PTH

Commit message: Updated board to fix a number of problems
* Used DMN53D0LW layout for the DMN6140L part which has a smaller footprint. Created a new layout for DMN6140L and used that
* Removed resistor in series with flyback diode.
* Updated diode layout to be 1N4004 compatible
* Removed diode across FET (was there assuming it would be a BJT)
* Fixed reset resistor, attaching it to VCC rather than GND
* Added a cap from reset to ground
* Fixed motor PWM output pin from ADC6 (not for pwm output) to ADC0
Parts:
- removed D1: (no value), SparkFun:DIODEPTH
- removed MOTOR-BAD_FOOTPRINT: DMN53D0LW, GARTH:DMN53D0LW
- removed R1: (no value), SparkFun:RESISTOR1206
- added D2: 1N4004, diode:1N4004
- U$2: value DIODE-ZENERPTH -> DMN6140L; device SparkFun:DIODE-ZENERPTH -> GARTH:DMN6140L
Connections:
- removed net N$1: D1.A, R1.2
- removed net V5: R3.1
- net 12V: now also D2.C; no longer D1.C
- net 5V: now also R3.1
- net GND: now also U$2.S; no longer MOTOR-BAD_FOOTPRINT.S, U$2.A
- net MOTOR-: now also D2.A, U$2.D; no longer MOTOR-BAD_FOOTPRINT.D, R1.1, U$2.C
- net MOTOR_CTRL: now also U$2.G; no longer MOTOR-BAD_FOOTPRINT.G
